Commit message: It launches without errors, but there is no planning

File: annin_ar4_description/urdf/ar.ros2_control.xacro (robot description, xacro)
@@ -2,5 +2,4 @@
 <robot xmlns:xacro="http://www.ros.org/wiki/xacro">
   <xacro:macro name="ar_ros2_control" params="
-    ar_model
     plugin_name
     serial_port
@@ -9,5 +8,4 @@
     joint_offset_parameters_file
     driver_parameters_file
-    tf_prefix
   ">
     <xacro:property name="robot_parameters"
@@ -17,15 +15,13 @@
     <xacro:property name="driver_parameters"
       value="${xacro.load_yaml(driver_parameters_file)}"/>
-    <ros2_control name="${ar_model}" type="system">
+    <ros2_control name="ar_controller" type="system">
       <hardware>
         <plugin>${plugin_name}</plugin>
-        <param name="ar_model">${ar_model}</param>
         <param name="serial_port">${serial_port}</param>
         <param name="calibrate">${calibrate}</param>
         <param name="calib_sequence">${driver_parameters['calib_sequence']}</param>
         <param name="velocity_control_enabled">${driver_parameters['velocity_control_enabled']}</param>
-        <param name="tf_prefix">${tf_prefix}</param>
       </hardware>
-      <joint name="${tf_prefix}joint_1">
+      <joint name="joint_1">
         <command_interface name="position">
           <param name="min">${robot_parameters['j1_limit_min']}</param>
@@ -41,5 +37,5 @@
         <param name="position_offset">${joint_offset_parameters['joint_1']}</param>
       </joint>
-      <joint name="${tf_prefix}joint_2">
+      <joint name="joint_2">
         <command_interface name="position">
           <param name="min">${robot_parameters['j2_limit_min']}</param>
@@ -55,5 +51,5 @@
         <param name="position_offset">${joint_offset_parameters['joint_2']}</param>
       </joint>
-      <joint name="${tf_prefix}joint_3">
+      <joint name="joint_3">
         <command_interface name="position">
           <param name="min">${robot_parameters['j3_limit_min']}</param>
@@ -69,5 +65,5 @@
         <param name="position_offset">${joint_offset_parameters['joint_3']}</param>
       </joint>
-      <joint name="${tf_prefix}joint_4">
+      <joint name="joint_4">
         <command_interface name="position">
           <param name="min">${robot_parameters['j4_limit_min']}</param>
@@ -83,5 +79,5 @@
         <param name="position_offset">${joint_offset_parameters['joint_4']}</param>
       </joint>
-      <joint name="${tf_prefix}joint_5">
+      <joint name="joint_5">
         <command_interface name="position">
           <param name="min">${robot_parameters['j5_limit_min']}</param>
@@ -97,5 +93,5 @@
         <param name="position_offset">${joint_offset_parameters['joint_5']}</param>
       </joint>
-      <joint name="${tf_prefix}joint_6">
+      <joint name="joint_6">
         <command_interface name="position">
           <param name="min">${robot_parameters['j6_limit_min']}</param>

File: annin_ar4_description/urdf/ar.urdf.xacro (robot description, xacro)
@@ -1,12 +1,10 @@
 <?xml version="1.0"?>
-<robot xmlns:xacro="http://wiki.ros.org/xacro" name="$(arg ar_model)">
-  <xacro:arg name="tf_prefix" default="" />
-  <xacro:arg name="include_gripper" default="true"/>
+<robot xmlns:xacro="http://wiki.ros.org/xacro" name="ar_robot">
+  <xacro:arg name="include_gripper" default="false"/>
   <xacro:include filename="$(find annin_ar4_description)/urdf/ar_macro.xacro"/>
   <link name="world" />
   <xacro:ar_robot
-    tf_prefix="$(arg tf_prefix)"
     parent="world"
-    robot_parameters_file="$(find annin_ar4_description)/config/$(arg ar_model).yaml"
+    robot_parameters_file="$(find annin_ar4_description)/config/mk2.yaml"
   >
     <origin xyz="0 0 0" rpy="0 0 0" />
@@ -15,6 +13,5 @@
     <xacro:include filename="$(find annin_ar4_description)/urdf/ar_gripper_macro.xacro"/>
     <xacro:ar_gripper
-      tf_prefix="$(arg tf_prefix)"
-      parent="$(arg tf_prefix)ee_link"
+      parent="ee_link"
     />
   </xacro:if>

File: annin_ar4_description/urdf/ar_gripper.ros2_control.xacro (robot description, xacro)
@@ -5,5 +5,4 @@
     plugin_name
     serial_port
-    tf_prefix
   ">
     <ros2_control name="${name}" type="system">
@@ -11,7 +10,6 @@
         <plugin>${plugin_name}</plugin>
         <param name="serial_port">${serial_port}</param>
-        <param name="tf_prefix">${tf_prefix}</param>
       </hardware>
-      <joint name="${tf_prefix}gripper_jaw1_joint">
+      <joint name="gripper_jaw1_joint">
         <command_interface name="position" />
         <state_interface name="position">
@@ -22,6 +20,6 @@
         </state_interface>
       </joint>
-      <joint name="${tf_prefix}gripper_jaw2_joint">
-        <param name="mimic">${tf_prefix}gripper_jaw1_joint</param>
+      <joint name="gripper_jaw2_joint">
+        <param name="mimic">gripper_jaw1_joint</param>
         <param name="multiplier">1</param>
         <state_interface name="position">

File: annin_ar4_description/urdf/ar_gripper_macro.xacro (robot description, xacro)
@@ -2,13 +2,12 @@
 <robot xmlns:xacro="http://wiki.ros.org/xacro">
   <xacro:macro name="ar_gripper" params="
-    tf_prefix
     parent
   ">
-    <joint name="${tf_prefix}gripper_base_joint" type="fixed">
+    <joint name="gripper_base_joint" type="fixed">
       <origin xyz="0.0 0.0 0.0" rpy="-1.5708 0.0 0.0"/>
       <parent link="${parent}"/>
-      <child link="${tf_prefix}gripper_base_link"/>
+      <child link="gripper_base_link"/>
     </joint>
-    <link name="${tf_prefix}gripper_base_link">
+    <link name="gripper_base_link">
       <visual>
         <geometry>
@@ -30,5 +29,5 @@
       </inertial>
     </link>
-    <link name="${tf_prefix}gripper_jaw1_link">
+    <link name="gripper_jaw1_link">
       <visual>
         <geometry>
@@ -50,5 +49,5 @@
       </inertial>
     </link>
-    <link name="${tf_prefix}gripper_jaw2_link">
+    <link name="gripper_jaw2_link">
       <visual>
         <geometry>
@@ -70,18 +69,18 @@
       </inertial>
     </link>
-    <joint name="${tf_prefix}gripper_jaw1_joint" type="prismatic">
+    <joint name="gripper_jaw1_joint" type="prismatic">
       <origin xyz="0.0 -0.036 0" rpy="0.0 0.0 0.0"/>
-      <parent link="${tf_prefix}gripper_base_link"/>
-      <child link="${tf_prefix}gripper_jaw1_link"/>
+      <parent link="gripper_base_link"/>
+      <child link="gripper_jaw1_link"/>
       <axis xyz="-1 0 0"/>
       <limit lower="0" upper="0.014" effort="-1" velocity="1.0"/>
     </joint>
-    <joint name="${tf_prefix}gripper_jaw2_joint" type="prismatic">
+    <joint name="gripper_jaw2_joint" type="prismatic">
       <origin xyz="0.0 -0.036 0" rpy="0.0 ${-pi} 0.0"/>
-      <parent link="${tf_prefix}gripper_base_link"/>
-      <child link="${tf_prefix}gripper_jaw2_link"/>
+      <parent link="gripper_base_link"/>
+      <child link="gripper_jaw2_link"/>
       <axis xyz="-1 0 0"/>
       <limit lower="0" upper="0.014" effort="1000" velocity="1.0"/>
-      <mimic joint="${tf_prefix}gripper_jaw1_joint" multiplier="1" offset="0"/>
+      <mimic joint="gripper_jaw1_joint" multiplier="1" offset="0"/>
     </joint>
   </xacro:macro>

File: annin_ar4_description/urdf/ar_macro.xacro (robot description, xacro)
@@ -1,6 +1,5 @@
 <?xml version="1.0" encoding="utf-8"?>
 <robot xmlns:xacro="http://wiki.ros.org/xacro">
-  <xacro:macro name="ar_robot" params="
-    tf_prefix
+  <xacro:macro name="ar_manipulator" params="
     parent
     *origin
@@ -8,10 +7,10 @@
   ">
     <xacro:property name="robot_parameters" value="${xacro.load_yaml(robot_parameters_file)}"/>
-    <joint name="${tf_prefix}base_joint" type="fixed">
+    <joint name="base_joint" type="fixed">
       <xacro:insert_block name="origin" />
       <parent link="${parent}"/>
-      <child link="${tf_prefix}base_link" />
-    </joint>
-    <link name="${tf_prefix}base_link">
+      <child link="base_link" />
+    </joint>
+    <link name="base_link">
       <inertial>
         <origin rpy="0 0 0" xyz="-4.6941E-06 0.054174 0.038824"/>
@@ -35,5 +34,5 @@
       </collision>
     </link>
-    <link name="${tf_prefix}link_1">
+    <link name="link_1">
       <inertial>
         <origin rpy="0 0 0" xyz="-0.022706 0.04294 -0.12205"/>
@@ -57,8 +56,8 @@
       </collision>
     </link>
-    <joint name="${tf_prefix}joint_1" type="revolute">
+    <joint name="joint_1" type="revolute">
       <origin rpy="${pi} 0 0" xyz="0 0 0"/>
-      <parent link="${tf_prefix}base_link"/>
-      <child link="${tf_prefix}link_1"/>
+      <parent link="base_link"/>
+      <child link="link_1"/>
       <axis xyz="0 0 1"/>
       <limit
@@ -69,5 +68,5 @@
       />
     </joint>
-    <link name="${tf_prefix}link_2">
+    <link name="link_2">
       <inertial>
         <origin rpy="0 0 0" xyz="0.064818 -0.11189 -0.038671"/>
@@ -91,8 +90,8 @@
       </collision>
     </link>
-    <joint name="${tf_prefix}joint_2" type="revolute">
+    <joint name="joint_2" type="revolute">
       <origin rpy="1.5708 0 -1.5708" xyz="0 0.0642 -0.16977"/>
-      <parent link="${tf_prefix}link_1"/>
-      <child link="${tf_prefix}link_2"/>
+      <parent link="link_1"/>
+      <child link="link_2"/>
       <axis xyz="0 0 -1"/>
       <limit
@@ -103,5 +102,5 @@
       />
     </joint>
-    <link name="${tf_prefix}link_3">
+    <link name="link_3">
       <inertial>
         <origin rpy="0 0 0" xyz="-0.00029765 -0.023661 -0.0019125"/>
@@ -125,8 +124,8 @@
       </collision>
     </link>
-    <joint name="${tf_prefix}joint_3" type="revolute">
+    <joint name="joint_3" type="revolute">
       <origin rpy="0 0 3.1416" xyz="0 -0.305 0.007"/>
-      <parent link="${tf_prefix}link_2"/>
-      <child link="${tf_prefix}link_3"/>
+      <parent link="link_2"/>
+      <child link="link_3"/>
       <axis xyz="0 0 -1"/>
       <limit
@@ -137,5 +136,5 @@
       />
     </joint>
-    <link name="${tf_prefix}link_4">
+    <link name="link_4">
       <inertial>
         <origin rpy="0 0 0" xyz="-0.0016798 -0.00057319 -0.074404"/>
@@ -159,8 +158,8 @@
       </collision>
     </link>
-    <joint name="${tf_prefix}joint_4" type="revolute">
+    <joint name="joint_4" type="revolute">
       <origin rpy="1.5708 0 -1.5708" xyz="0 0 0.0"/>
-      <parent link="${tf_prefix}link_3"/>
-      <child link="${tf_prefix}link_4"/>
+      <parent link="link_3"/>
+      <child link="link_4"/>
       <axis xyz="0 0 -1"/>
       <limit
@@ -171,5 +170,5 @@
       />
     </joint>
-    <link name="${tf_prefix}link_5">
+    <link name="link_5">
       <inertial>
         <origin rpy="0 0 0" xyz="0.0015066 -1.3102E-05 -0.012585"/>
@@ -193,8 +192,8 @@
       </collision>
     </link>
-    <joint name="${tf_prefix}joint_5" type="revolute">
+    <joint name="joint_5" type="revolute">
       <origin rpy="${pi} 0 -1.5708" xyz="0 0 -0.22263"/>
-      <parent link="${tf_prefix}link_4"/>
-      <child link="${tf_prefix}link_5"/>
+      <parent link="link_4"/>
+      <child link="link_5"/>
       <axis xyz="1 0 0"/>
       <limit
@@ -205,5 +204,5 @@
       />
     </joint>
-    <link name="${tf_prefix}link_6">
+    <link name="link_6">
       <inertial>
         <origin rpy="0 0 0" xyz="2.9287E-10 -1.6472E-09 0.0091432"/>
@@ -227,8 +226,8 @@
       </collision>
     </link>
-    <joint name="${tf_prefix}joint_6" type="revolute">
+    <joint name="joint_6" type="revolute">
       <origin rpy="0 0 3.1416" xyz="0.000 0 ${robot_parameters['l6_length']}"/>
-      <parent link="${tf_prefix}link_5"/>
-      <child link="${tf_prefix}link_6"/>
+      <parent link="link_5"/>
+      <child link="link_6"/>
       <axis xyz="0 0 1"/>
       <limit
@@ -240,8 +239,8 @@
     </joint>
     <!-- center of the end effector mounting surface on link_6 -->
-    <link name="${tf_prefix}ee_link" />
-    <joint name="${tf_prefix}ee_joint" type="fixed">
-      <parent link="${tf_prefix}link_6" />
-      <child link="${tf_prefix}ee_link" />
+    <link name="ee_link" />
+    <joint name="ee_joint" type="fixed">
+      <parent link="link_6" />
+      <child link="ee_link" />
       <origin xyz="0 0 0.0" rpy="0 0 0" />
     </joint>

File: annin_ar4_driver/urdf/ar.urdf.xacro (robot description, xacro)
@@ -1,28 +1,25 @@
 <?xml version="1.0"?>
-<robot xmlns:xacro="http://wiki.ros.org/xacro" name="$(arg ar_model)">
+<robot xmlns:xacro="http://wiki.ros.org/xacro" name="ar_robot">
   <xacro:arg name="serial_port" default="/dev/ttyACM0"/>
   <xacro:arg name="arduino_serial_port" default="/dev/ttyUSB0"/>
   <xacro:arg name="calibrate" default="True"/>
-  <xacro:arg name="tf_prefix" default="" />
-  <xacro:arg name="include_gripper" default="true"/>
+  <xacro:arg name="include_gripper" default="false"/>
   <xacro:include filename="$(find annin_ar4_description)/urdf/ar_macro.xacro"/>
   <xacro:include filename="$(find annin_ar4_description)/urdf/ar.ros2_control.xacro"/>
   <link name="world" />
   <xacro:ar_robot
-    tf_prefix="$(arg tf_prefix)"
     parent="world"
-    robot_parameters_file="$(find annin_ar4_description)/config/$(arg ar_model).yaml"
+    robot_parameters_file="$(find annin_ar4_description)/config/mk2.yaml"
   >
     <origin xyz="0 0 0" rpy="0 0 0" />
   </xacro:ar_robot>
   <xacro:ar_ros2_control
-    ar_model="$(arg ar_model)"
+    ar_model="mk2"
     plugin_name="annin_ar4_driver/ARHardwareInterface"
     serial_port="$(arg serial_port)"
     calibrate="$(arg calibrate)"
-    robot_parameters_file="$(find annin_ar4_description)/config/$(arg ar_model).yaml"
-    joint_offset_parameters_file="$(find annin_ar4_driver)/config/joint_offsets/$(arg ar_model).yaml"
+    robot_parameters_file="$(find annin_ar4_description)/config/mk2.yaml"
+    joint_offset_parameters_file="$(find annin_ar4_driver)/config/joint_offsets/mk2.yaml"
     driver_parameters_file="$(find annin_ar4_driver)/config/driver.yaml"
-    tf_prefix="$(arg tf_prefix)"
   />
   <xacro:if value="$(arg include_gripper)">
@@ -30,6 +27,5 @@
     <xacro:include filename="$(find annin_ar4_description)/urdf/ar_gripper.ros2_control.xacro"/>
     <xacro:ar_gripper
-      tf_prefix="$(arg tf_prefix)"
-      parent="$(arg tf_prefix)ee_link"
+      parent="ee_link"
     />
     <xacro:ar_gripper_ros2_control
@@ -37,5 +33,4 @@
       plugin_name="annin_ar4_driver/ARServoGripperHWInterface"
       serial_port="$(arg arduino_serial_port)"
-      tf_prefix="$(arg tf_prefix)"
     />
   </xacro:if>

File: annin_ar4_moveit_config/srdf/ar.srdf.xacro (robot description, xacro)
@@ -1,11 +1,8 @@
 <?xml version="1.0" encoding="UTF-8"?>
-<robot xmlns:xacro="http://wiki.ros.org/xacro" name="$(arg name)">
-  <xacro:arg name="include_gripper" default="true"/>
-  <xacro:arg name="tf_prefix" default="" />
+<robot xmlns:xacro="http://wiki.ros.org/xacro" name="ar_robot">
+  <xacro:arg name="include_gripper" default="false"/>
   <xacro:include filename="$(find annin_ar4_moveit_config)/srdf/ar_macro.srdf.xacro"/>
-  <xacro:ar_srdf tf_prefix="$(arg tf_prefix)"/>
   <xacro:if value="$(arg include_gripper)">
     <xacro:include filename="$(find annin_ar4_moveit_config)/srdf/ar_gripper_macro.srdf.xacro"/>
-    <xacro:ar_gripper_srdf tf_prefix="$(arg tf_prefix)"/>
   </xacro:if>
 </robot>

File: annin_ar4_moveit_config/srdf/ar_gripper_macro.srdf.xacro (robot description, xacro)
@@ -5,23 +5,23 @@
 -->
 <robot xmlns:xacro="http://wiki.ros.org/xacro">
-  <xacro:macro name="ar_gripper_srdf" params="tf_prefix">
+  <xacro:macro name="ar_gripper_srdf">
     <group name="ar_gripper">
-      <link name="${tf_prefix}gripper_base_link" />
-      <link name="${tf_prefix}gripper_jaw1_link" />
-      <link name="${tf_prefix}gripper_jaw2_link" />
-      <joint name="${tf_prefix}gripper_jaw1_joint" />
-      <passive_joint name="${tf_prefix}gripper_jaw2_joint" />
+      <link name="gripper_base_link" />
+      <link name="gripper_jaw1_link" />
+      <link name="gripper_jaw2_link" />
+      <joint name="gripper_jaw1_joint" />
+      <passive_joint name="gripper_jaw2_joint" />
     </group>
     <group_state name="open" group="ar_gripper">
-      <joint name="${tf_prefix}gripper_jaw1_joint" value="0.012" />
+      <joint name="gripper_jaw1_joint" value="0.012" />
     </group_state>
     <group_state name="closed" group="ar_gripper">
-      <joint name="${tf_prefix}gripper_jaw1_joint" value="0.001" />
+      <joint name="gripper_jaw1_joint" value="0.001" />
     </group_state>
-    <disable_collisions link1="${tf_prefix}gripper_base_link" link2="${tf_prefix}gripper_jaw1_link" reason="Adjacent" />
-    <disable_collisions link1="${tf_prefix}gripper_base_link" link2="${tf_prefix}gripper_jaw2_link" reason="Adjacent" />
-    <disable_collisions link1="${tf_prefix}gripper_jaw1_link" link2="${tf_prefix}gripper_jaw2_link" reason="Default" />
-    <disable_collisions link1="${tf_prefix}link_6" link2="${tf_prefix}gripper_base_link" reason="Adjacent" />
-    <disable_collisions link1="${tf_prefix}link_5" link2="${tf_prefix}gripper_base_link" reason="Adjacent" />
+    <disable_collisions link1="gripper_base_link" link2="gripper_jaw1_link" reason="Adjacent" />
+    <disable_collisions link1="gripper_base_link" link2="gripper_jaw2_link" reason="Adjacent" />
+    <disable_collisions link1="gripper_jaw1_link" link2="gripper_jaw2_link" reason="Default" />
+    <disable_collisions link1="link_6" link2="gripper_base_link" reason="Adjacent" />
+    <disable_collisions link1="link_5" link2="gripper_base_link" reason="Adjacent" />
   </xacro:macro>
 </robot>

File: annin_ar4_moveit_config/srdf/ar_macro.srdf.xacro (robot description, xacro)
@@ -5,39 +5,39 @@
 -->
 <robot xmlns:xacro="http://wiki.ros.org/xacro">
-  <xacro:macro name="ar_srdf" params="tf_prefix">
+  <xacro:macro name="ar_robot">
     <group name="ar_manipulator">
-      <joint name="${tf_prefix}joint_1" />
-      <joint name="${tf_prefix}joint_2" />
-      <joint name="${tf_prefix}joint_3" />
-      <joint name="${tf_prefix}joint_4" />
-      <joint name="${tf_prefix}joint_5" />
-      <joint name="${tf_prefix}joint_6" />
-      <joint name="${tf_prefix}ee_joint"/>
+      <joint name="joint_1" />
+      <joint name="joint_2" />
+      <joint name="joint_3" />
+      <joint name="joint_4" />
+      <joint name="joint_5" />
+      <joint name="joint_6" />
+      <joint name="ee_joint"/>
     </group>
     <group_state name="home" group="ar_manipulator">
-      <joint name="${tf_prefix}joint_1" value="0" />
-      <joint name="${tf_prefix}joint_2" value="0" />
-      <joint name="${tf_prefix}joint_3" value="0" />
-      <joint name="${tf_prefix}joint_4" value="0" />
-      <joint name="${tf_prefix}joint_5" value="0" />
-      <joint name="${tf_prefix}joint_6" value="0" />
+      <joint name="joint_1" value="0" />
+      <joint name="joint_2" value="0" />
+      <joint name="joint_3" value="0" />
+      <joint name="joint_4" value="0" />
+      <joint name="joint_5" value="0" />
+      <joint name="joint_6" value="0" />
     </group_state>
     <group_state name="upright" group="ar_manipulator">
-      <joint name="${tf_prefix}joint_1" value="0" />
-      <joint name="${tf_prefix}joint_2" value="-0.087" />
-      <joint name="${tf_prefix}joint_3" value="-1.4" />
-      <joint name="${tf_prefix}joint_4" value="0" />
-      <joint name="${tf_prefix}joint_5" value="0" />
-      <joint name="${tf_prefix}joint_6" value="0" />
+      <joint name="joint_1" value="0" />
+      <joint name="joint_2" value="-0.087" />
+      <joint name="joint_3" value="-1.4" />
+      <joint name="joint_4" value="0" />
+      <joint name="joint_5" value="0" />
+      <joint name="joint_6" value="0" />
     </group_state>
-    <disable_collisions link1="${tf_prefix}base_link" link2="${tf_prefix}link_1" reason="Adjacent" />
-    <disable_collisions link1="${tf_prefix}link_1" link2="${tf_prefix}link_2" reason="Adjacent" />
-    <disable_collisions link1="${tf_prefix}link_1" link2="${tf_prefix}link_3" reason="Never" />
-    <disable_collisions link1="${tf_prefix}link_2" link2="${tf_prefix}link_3" reason="Adjacent" />
-    <disable_collisions link1="${tf_prefix}link_3" link2="${tf_prefix}link_4" reason="Adjacent" />
-    <disable_collisions link1="${tf_prefix}link_3" link2="${tf_prefix}link_5" reason="Never" />
-    <disable_collisions link1="${tf_prefix}link_3" link2="${tf_prefix}link_6" reason="Never" />
-    <disable_collisions link1="${tf_prefix}link_4" link2="${tf_prefix}link_5" reason="Adjacent" />
-    <disable_collisions link1="${tf_prefix}link_5" link2="${tf_prefix}link_6" reason="Adjacent" />
+    <disable_collisions link1="base_link" link2="link_1" reason="Adjacent" />
+    <disable_collisions link1="link_1" link2="link_2" reason="Adjacent" />
+    <disable_collisions link1="link_1" link2="link_3" reason="Never" />
+    <disable_collisions link1="link_2" link2="link_3" reason="Adjacent" />
+    <disable_collisions link1="link_3" link2="link_4" reason="Adjacent" />
+    <disable_collisions link1="link_3" link2="link_5" reason="Never" />
+    <disable_collisions link1="link_3" link2="link_6" reason="Never" />
+    <disable_collisions link1="link_4" link2="link_5" reason="Adjacent" />
+    <disable_collisions link1="link_5" link2="link_6" reason="Adjacent" />
   </xacro:macro>
 </robot>

File: annin_ar4_moveit_config/urdf/fake_ar.urdf.xacro (robot description, xacro)
@@ -1,30 +1,25 @@
 <?xml version="1.0"?>
-<robot xmlns:xacro="http://wiki.ros.org/xacro" name="$(arg ar_model)">
+<robot xmlns:xacro="http://wiki.ros.org/xacro" name="ar_robot">
   <xacro:include filename="$(find annin_ar4_description)/urdf/ar_macro.xacro"/>
   <xacro:include filename="$(find annin_ar4_description)/urdf/ar_gripper_macro.xacro"/>
   <xacro:include filename="$(find annin_ar4_description)/urdf/ar.ros2_control.xacro"/>
   <xacro:include filename="$(find annin_ar4_description)/urdf/ar_gripper.ros2_control.xacro"/>
-  <xacro:arg name="tf_prefix" default="" />
   <link name="world" />
-  <xacro:ar_robot
-    tf_prefix="$(arg tf_prefix)"
+  <xacro:ar_manipulator
     parent="world"
-    robot_parameters_file="$(find annin_ar4_description)/config/$(arg ar_model).yaml"
+    robot_parameters_file="$(find annin_ar4_description)/config/mk2.yaml"
   >
     <origin xyz="0 0 0" rpy="0 0 0" />
-  </xacro:ar_robot>
+  </xacro:ar_manipulator>
   <xacro:ar_gripper
-    tf_prefix="$(arg tf_prefix)"
-    parent="$(arg tf_prefix)ee_link"
+    parent="ee_link"
   />
   <xacro:ar_ros2_control
-    ar_model="$(arg ar_model)"
     plugin_name="mock_components/GenericSystem"
     serial_port="/dev/ttyACM0"
     calibrate="False"
-    robot_parameters_file="$(find annin_ar4_description)/config/$(arg ar_model).yaml"
-    joint_offset_parameters_file="$(find annin_ar4_driver)/config/joint_offsets/$(arg ar_model).yaml"
+    robot_parameters_file="$(find annin_ar4_description)/config/mk2.yaml"
+    joint_offset_parameters_file="$(find annin_ar4_driver)/config/joint_offsets/mk2.yaml"
     driver_parameters_file="$(find annin_ar4_driver)/config/driver.yaml"
-    tf_prefix="$(arg tf_prefix)"
   />
   <xacro:ar_gripper_ros2_control
@@ -32,5 +27,4 @@
     plugin_name="mock_components/GenericSystem"
     serial_port="/dev/ttyUSB0"
-    tf_prefix="$(arg tf_prefix)"
   />
 </robot>
