Commit message: Servoing now works

File: gorm_arm/urdf/fake_gorm_arm.urdf (robot description, URDF)
Before this commit: robot gorm_arm, 9 links, 8 joints
Joints:
- joint joint_1: limit lower=-150 upper=184 effort=-1 velocity=1.0472 -> lower=-2.618 upper=3.2114 effort=-1 velocity=1.0472
- joint joint_2: limit lower=-47 upper=120 effort=-1 velocity=1.0472 -> lower=-0.8203 upper=2.0944 effort=-1 velocity=1.0472
- joint joint_3: limit lower=-110 upper=62 effort=-1 velocity=1.0472 -> lower=-1.9199 upper=1.0821 effort=-1 velocity=1.0472
- joint joint_4: limit lower=-177 upper=161 effort=-1 velocity=1.0472 -> lower=-3.0892 upper=2.81 effort=-1 velocity=1.0472
- joint joint_5: limit lower=-103 upper=103 effort=-1 velocity=1.0472 -> lower=-1.7977 upper=1.7977 effort=-1 velocity=1.0472; origin xyz=0 0 -0.22263 rpy=${pi} 0 -1.5708 -> xyz=0 0 -0.22263 rpy=3 0 -1.5708
- joint joint_6: limit lower=-167 upper=170 effort=-1 velocity=1.0472 -> lower=-2.9147 upper=2.9671 effort=-1 velocity=1.0472

Commit message: Fixed urdf lenghts, but not mesh

File: gorm_arm/urdf/fake_gorm_arm.urdf (robot description, URDF)
Before this commit: robot gorm_arm, 9 links, 8 joints
Joints:
- joint joint_3: origin xyz=0 -0.305 0.007 rpy=0 0 3.1416 -> xyz=0 -0.34997 0.0046 rpy=0 0 3.1416
- joint joint_5: origin xyz=0 0 -0.22263 rpy=3 0 -1.5708 -> xyz=0 0 -0.27435 rpy=3.1416 0 -1.5708
