Commit message: Added the 40 deg angle to the urdf

File: gorm_arm/urdf/gorm_arm_horiz.urdf (robot description, URDF)
Before this commit: robot gorm_arm, 9 links, 8 joints
Joints:
- joint base_joint: origin xyz=0 0 0 rpy=0.6981 0 0 -> (none)
- joint joint_1: origin xyz=0 0 0 rpy=${pi} 0 0.5236 -> xyz=0 0 0 rpy=${pi} 0 0
