Commit message: changed README

File: gorm_arm/urdf/gorm_arm.urdf (robot description, URDF)
Before this commit: robot gorm_arm, 9 links, 8 joints
Joints:
- joint joint_1: limit lower=-2.618 upper=3.2114 effort=-1 velocity=1.0472 -> lower=-3.2114 upper=2.618 effort=-1 velocity=1.0472

Commit message: stable commit

File: gorm_arm/urdf/gorm_arm.urdf (robot description, URDF)
Before this commit: robot gorm_arm, 9 links, 8 joints
Joints:
- joint base_joint: origin (none) -> xyz=0 0 0 rpy=0.6981 0 0
- joint joint_1: origin xyz=0 0 0 rpy=${pi} 0 0 -> xyz=0 0 0 rpy=${pi} 0 0.5236
